File: hardware/schematics and pcb/amplifier.kicad_pcb (KiCad board)
At the start: 2 copper layers, 99.1 x 99.1 mm, 73 parts, among them J1 JACK_2P, P1 CONN_01X03, P2 CONN_01X07, P3 CONN_01X07, P4 CONN_01X20, P5 CONN_01X20, P6 CONN_01X20, P7 CONN_01X20, P8 CONN_01X02, SW1 Switch_DPST, U1 AD620, U2 LM324, U3 MCP3008, U4 CA3140

Commit message: fixed a couple of things in the pcb and added 3d models
Parts:
- added P10: CONN_01X04, Pin_Headers:Pin_Header_Straight_1x04, F.Cu at (154.3, 64.8)
- added P9: CONN_01X02, Pin_Headers:Pin_Header_Straight_1x02, F.Cu at (91.4, 121.9)
- R12: value 470K -> 890K
- R13: value 470K -> 1.8
- R17: value 470K -> .6
- R19: value 10K -> 15K
- R20: value 15K -> 10K
- R21: value 1K -> 10
- R5, R6: value 100 -> 220
- moved R14 6.38 mm to (149.2, 76.2)
- moved R16 6.38 mm to (159.4, 82.5)
- moved R17 6.38 mm to (149.2, 69.8)
Connections:
- P6 pad 7: Net-(P5-Pad5) -> Net-(P6-Pad7)
- R21 pad 2: Net-(P6-Pad8) -> Net-(P7-Pad16)
- R22 pad 1: Net-(P7-Pad7) -> Net-(P7-Pad8)
Routing:
- net Net-(P7-Pad8): track 0.00 -> 145.6 mm, vias 0 -> 3
- net Net-(P7-Pad16): track 0.00 -> 52.9 mm, vias 0 -> 2
- net VEE: track 312.3 -> 338.3 mm, vias 3 -> 5
- net Net-(P6-Pad7): track 0.00 -> 19.4 mm, vias 0 -> 1
- net Net-(P5-Pad5): track 110.8 -> 91.4 mm, vias 2 -> 1
- net Net-(P6-Pad8): track 85.3 -> 73.8 mm
- net Net-(C21-Pad1): track 114.7 -> 121.1 mm
- net Net-(C18-Pad2): track 36.7 -> 30.7 mm
- net Net-(C21-Pad2): track 45.9 -> 51.0 mm
- net Net-(R15-Pad1): track 60.6 -> 56.0 mm, vias 0 -> 2
- net Net-(P7-Pad7): track 79.0 -> 76.5 mm
- net Net-(C17-Pad1): track 60.3 -> 61.5 mm

Commit message: more fixes in the pcb
Routing:
- net Net-(P6-Pad8): track 73.8 -> 0.00 mm
- net Net-(P7-Pad7): track 76.5 -> 18.1 mm, vias 2 -> 0
- net Net-(P6-Pad7): track 19.4 -> 0.00 mm, vias 1 -> 0
- net Net-(P5-Pad5): track 91.4 -> 78.6 mm, vias 1 -> 0
- net Net-(P7-Pad16): track 52.9 -> 41.5 mm
- net Net-(P7-Pad8): track 145.6 -> 143.1 mm
